File: pcb/my-keyboard.kicad_pcb (KiCad board)
At the start: 2 copper layers, 86.5 x 59.5 mm, 12 parts, among them J2 Conn_01x04, SW1 SW_Push, SW2 SW_Push, SW3 SW_Push, SW4 SW_Push, SW7 RotaryEncoder_Switch, SW8 RotaryEncoder_Switch, U1 MOUDLE-SEEEDUINO-XIAO

Commit message: Added cad models
Parts:
- added REF**: MountingHole_2.2mm_M2, MountingHole:MountingHole_2.2mm_M2, F.Cu at (136.5, 73.0)
- added REF**: MountingHole_2.2mm_M2, MountingHole:MountingHole_2.2mm_M2, F.Cu at (101.0, 117.0)
- added REF**: MountingHole_2.2mm_M2, MountingHole:MountingHole_2.2mm_M2, F.Cu at (178.5, 90.5)
- added REF**: MountingHole_2.2mm_M2, MountingHole:MountingHole_2.2mm_M2, F.Cu at (101.0, 63.5)
Other:
- board size 86.5 x 59.5 mm -> 90.5 x 60.5 mm
