File: pcb/my-keyboard.kicad_pcb (KiCad board)
At the start: 2 copper layers, 90.5 x 60.5 mm, 16 parts, among them J2 Conn_01x04, SW1 SW_Push, SW2 SW_Push, SW3 SW_Push, SW4 SW_Push, SW7 RotaryEncoder_Switch, SW8 RotaryEncoder_Switch, U1 MOUDLE-SEEEDUINO-XIAO

Commit message: Added M3 mouting holes
Parts:
- removed the REF** at (136.5, 73.0)
- removed the REF** at (101.0, 117.0)
- removed the REF** at (178.5, 90.5)
- removed the REF** at (101.0, 63.5)
- added REF**: MountingHole_3.2mm_M3, MountingHole:MountingHole_3.2mm_M3, F.Cu at (101.0, 89.0)
- added REF**: MountingHole_3.2mm_M3, MountingHole:MountingHole_3.2mm_M3, F.Cu at (179.0, 88.0)
